File: pcb/matrix.kicad_sch (KiCad schematic)
At the start: 156 parts, among them SW10 F8, SW11 F9, SW12 F10, SW13 F11, SW14 F12, SW15 Help, SW16 Grv, SW17 1, SW18 2, SW19 3, SW2 Esc, SW20 4, SW21 5, SW22 6, SW23 7, SW24 8, SW25 9, SW26 0, SW27 -, SW28 =, SW29 Bksp, SW3 F1, SW30 Del, SW31 Tab, SW32 Q, SW33 W, SW34 E, SW35 R, SW36 T, SW37 Y, SW38 U, SW39 I, SW4 F2, SW40 O, SW41 P, SW42 [, SW43 ], SW44 \, SW45 Hyper, SW46 A, SW47 S, SW48 D, SW49 F, SW5 F3, SW50 G, SW51 H, SW52 J, SW53 K, SW54 L, SW55 ;, SW56 ', SW57 Enter, SW58 LShift, SW59 Z, SW6 F4, SW60 X, SW61 C, SW62 V, SW63 B, SW64 N, SW65 M, SW66 ,, SW67 ., SW68 /, SW69 RShift, SW7 F5, SW70 Up, SW71 Ctrl, SW72 LAlt, SW73 LAmiga, SW74 Space, SW75 RAmiga, SW76 RAlt, SW77 Left, SW78 Down, SW79 Right, SW8 F6, SW9 F7

Commit message: PCBs in the work
Parts:
- added D75: (no value), symbol Device:D_Small
- added SW75: (no value), symbol Switch:SW_Push
- D10, D11, D12, D13, D14, D15, D16, D17, D18, D19, D2, D20, D21, D22, D23, D24, D25, D26, D27, D28, D29, D3, D30, D31, D32, D33, D34, D35, D36, D37, D38, D39, D4, D40, D41, D42, D43, D44, D45, D46, D47, D48, D49, D5, D50, D51, D52, D53, D54, D55, D56, D57, D58, D59, D6, D60, D61, D62, D63, D64, D65, D66, D67, D68, D69, D7, D70, D71, D72, D73, D74, D8, D9: value D_Small -> (none); footprint Diode_SMD:D_SOD-123 -> (none)
- D76: renamed from D75; value D_Small -> (none); footprint Diode_SMD:D_SOD-123 -> (none)
- D77: renamed from D76; value D_Small -> (none); footprint Diode_SMD:D_SOD-123 -> (none)
- D78: renamed from D77; value D_Small -> (none); footprint Diode_SMD:D_SOD-123 -> (none)
- D79: renamed from D78; value D_Small -> (none); footprint Diode_SMD:D_SOD-123 -> (none)
- D80: renamed from D79; value D_Small -> (none); footprint Diode_SMD:D_SOD-123 -> (none)
- SW10: value F8 -> (none); footprint Button_Switch_Keyboard:SW_Cherry_MX_1.00u_PCB -> (none)
- SW11: value F9 -> (none); footprint Button_Switch_Keyboard:SW_Cherry_MX_1.00u_PCB -> (none)
- SW12: value F10 -> (none); footprint Button_Switch_Keyboard:SW_Cherry_MX_1.00u_PCB -> (none)
- SW13: value F11 -> (none); footprint Button_Switch_Keyboard:SW_Cherry_MX_1.00u_PCB -> (none)
- SW14: value F12 -> (none); footprint Button_Switch_Keyboard:SW_Cherry_MX_1.00u_PCB -> (none)
- SW15: value Help -> (none); footprint Button_Switch_Keyboard:SW_Cherry_MX_1.25u_PCB -> (none)
- SW16: value Grv -> (none); footprint Button_Switch_Keyboard:SW_Cherry_MX_1.00u_PCB -> (none)
- SW17: value 1 -> (none); footprint Button_Switch_Keyboard:SW_Cherry_MX_1.00u_PCB -> (none)
- SW18: value 2 -> (none); footprint Button_Switch_Keyboard:SW_Cherry_MX_1.00u_PCB -> (none)
- SW19: value 3 -> (none); footprint Button_Switch_Keyboard:SW_Cherry_MX_1.00u_PCB -> (none)
- SW2: value Esc -> (none); footprint Button_Switch_Keyboard:SW_Cherry_MX_1.25u_PCB -> (none)
- SW20: value 4 -> (none); footprint Button_Switch_Keyboard:SW_Cherry_MX_1.00u_PCB -> (none)
- SW21: value 5 -> (none); footprint Button_Switch_Keyboard:SW_Cherry_MX_1.00u_PCB -> (none)
- SW22: value 6 -> (none); footprint Button_Switch_Keyboard:SW_Cherry_MX_1.00u_PCB -> (none)
- SW23: value 7 -> (none); footprint Button_Switch_Keyboard:SW_Cherry_MX_1.00u_PCB -> (none)
- SW24: value 8 -> (none); footprint Button_Switch_Keyboard:SW_Cherry_MX_1.00u_PCB -> (none)
- SW25: value 9 -> (none); footprint Button_Switch_Keyboard:SW_Cherry_MX_1.00u_PCB -> (none)
- SW26: value 0 -> (none); footprint Button_Switch_Keyboard:SW_Cherry_MX_1.00u_PCB -> (none)
- SW27: value - -> (none); footprint Button_Switch_Keyboard:SW_Cherry_MX_1.00u_PCB -> (none)
- SW28: value = -> (none); footprint Button_Switch_Keyboard:SW_Cherry_MX_1.00u_PCB -> (none)
- SW29: value Bksp -> (none); footprint Button_Switch_Keyboard:SW_Cherry_MX_2.00u_PCB -> (none)
- SW3: value F1 -> (none); footprint Button_Switch_Keyboard:SW_Cherry_MX_1.00u_PCB -> (none)
- SW30: value Del -> (none); footprint Button_Switch_Keyboard:SW_Cherry_MX_1.00u_PCB -> (none)
- SW31: value Tab -> (none); footprint Button_Switch_Keyboard:SW_Cherry_MX_1.50u_PCB -> (none)
- SW32: value Q -> (none); footprint Button_Switch_Keyboard:SW_Cherry_MX_1.00u_PCB -> (none)
- SW33: value W -> (none); footprint Button_Switch_Keyboard:SW_Cherry_MX_1.00u_PCB -> (none)
- SW34: value E -> (none); footprint Button_Switch_Keyboard:SW_Cherry_MX_1.00u_PCB -> (none)
- SW35: value R -> (none); footprint Button_Switch_Keyboard:SW_Cherry_MX_1.00u_PCB -> (none)
- SW36: value T -> (none); footprint Button_Switch_Keyboard:SW_Cherry_MX_1.00u_PCB -> (none)
- SW37: value Y -> (none); footprint Button_Switch_Keyboard:SW_Cherry_MX_1.00u_PCB -> (none)
- SW38: value U -> (none); footprint Button_Switch_Keyboard:SW_Cherry_MX_1.00u_PCB -> (none)
- SW39: value I -> (none); footprint Button_Switch_Keyboard:SW_Cherry_MX_1.00u_PCB -> (none)
- SW4: value F2 -> (none); footprint Button_Switch_Keyboard:SW_Cherry_MX_1.00u_PCB -> (none)
- SW40: value O -> (none); footprint Button_Switch_Keyboard:SW_Cherry_MX_1.00u_PCB -> (none)
- SW41: value P -> (none); footprint Button_Switch_Keyboard:SW_Cherry_MX_1.00u_PCB -> (none)
- SW42: value [ -> (none); footprint Button_Switch_Keyboard:SW_Cherry_MX_1.00u_PCB -> (none)
- SW43: value ] -> (none); footprint Button_Switch_Keyboard:SW_Cherry_MX_1.00u_PCB -> (none)
- SW44: value \ -> (none); footprint Button_Switch_Keyboard:SW_Cherry_MX_1.50u_PCB -> (none)
- SW45: value Hyper -> (none); footprint Button_Switch_Keyboard:SW_Cherry_MX_2.00u_PCB -> (none)
- SW46: value A -> (none); footprint Button_Switch_Keyboard:SW_Cherry_MX_1.00u_PCB -> (none)
- SW47: value S -> (none); footprint Button_Switch_Keyboard:SW_Cherry_MX_1.00u_PCB -> (none)
- SW48: value D -> (none); footprint Button_Switch_Keyboard:SW_Cherry_MX_1.00u_PCB -> (none)
- SW49: value F -> (none); footprint Button_Switch_Keyboard:SW_Cherry_MX_1.00u_PCB -> (none)
- SW5: value F3 -> (none); footprint Button_Switch_Keyboard:SW_Cherry_MX_1.00u_PCB -> (none)
- SW50: value G -> (none); footprint Button_Switch_Keyboard:SW_Cherry_MX_1.00u_PCB -> (none)
- SW51: value H -> (none); footprint Button_Switch_Keyboard:SW_Cherry_MX_1.00u_PCB -> (none)
- SW52: value J -> (none); footprint Button_Switch_Keyboard:SW_Cherry_MX_1.00u_PCB -> (none)
- SW53: value K -> (none); footprint Button_Switch_Keyboard:SW_Cherry_MX_1.00u_PCB -> (none)
- SW54: value L -> (none); footprint Button_Switch_Keyboard:SW_Cherry_MX_1.00u_PCB -> (none)
- SW55: value ; -> (none); footprint Button_Switch_Keyboard:SW_Cherry_MX_1.00u_PCB -> (none)
- SW56: value ' -> (none); footprint Button_Switch_Keyboard:SW_Cherry_MX_1.00u_PCB -> (none)
- SW57: value Enter -> (none); footprint Button_Switch_Keyboard:SW_Cherry_MX_2.00u_PCB -> (none)
- SW58: value LShift -> (none); footprint Button_Switch_Keyboard:SW_Cherry_MX_1.75u_PCB -> (none)
- SW59: value Z -> (none); footprint Button_Switch_Keyboard:SW_Cherry_MX_1.00u_PCB -> (none)
- SW6: value F4 -> (none); footprint Button_Switch_Keyboard:SW_Cherry_MX_1.00u_PCB -> (none)
- SW60: value X -> (none); footprint Button_Switch_Keyboard:SW_Cherry_MX_1.00u_PCB -> (none)
- SW61: value C -> (none); footprint Button_Switch_Keyboard:SW_Cherry_MX_1.00u_PCB -> (none)
- SW62: value V -> (none); footprint Button_Switch_Keyboard:SW_Cherry_MX_1.00u_PCB -> (none)
- SW63: value B -> (none); footprint Button_Switch_Keyboard:SW_Cherry_MX_1.00u_PCB -> (none)
- SW64: value N -> (none); footprint Button_Switch_Keyboard:SW_Cherry_MX_1.00u_PCB -> (none)
- SW65: value M -> (none); footprint Button_Switch_Keyboard:SW_Cherry_MX_1.00u_PCB -> (none)
- SW66: value , -> (none); footprint Button_Switch_Keyboard:SW_Cherry_MX_1.00u_PCB -> (none)
- SW67: value . -> (none); footprint Button_Switch_Keyboard:SW_Cherry_MX_1.00u_PCB -> (none)
- SW68: value / -> (none); footprint Button_Switch_Keyboard:SW_Cherry_MX_1.00u_PCB -> (none)
- SW69: value RShift -> (none); footprint Button_Switch_Keyboard:SW_Cherry_MX_2.25u_PCB -> (none)
- SW7: value F5 -> (none); footprint Button_Switch_Keyboard:SW_Cherry_MX_1.00u_PCB -> (none)
- SW70: value Up -> (none); footprint Button_Switch_Keyboard:SW_Cherry_MX_1.00u_PCB -> (none)
- SW71: value Ctrl -> (none); footprint Button_Switch_Keyboard:SW_Cherry_MX_1.25u_PCB -> (none)
- SW72: value LAlt -> (none); footprint Button_Switch_Keyboard:SW_Cherry_MX_1.25u_PCB -> (none)
- SW73: value LAmiga -> (none); footprint Button_Switch_Keyboard:SW_Cherry_MX_1.25u_PCB -> (none)
- SW74: value Space -> (none); footprint Button_Switch_Keyboard:SW_Cherry_MX_6.25u_PCB -> (none)
- SW76: renamed from SW75; value RAmiga -> (none); footprint Button_Switch_Keyboard:SW_Cherry_MX_1.25u_PCB -> (none)
- SW77: renamed from SW76; value RAlt -> (none); footprint Button_Switch_Keyboard:SW_Cherry_MX_1.25u_PCB -> (none)
- SW78: renamed from SW77; value Left -> (none); footprint Button_Switch_Keyboard:SW_Cherry_MX_1.00u_PCB -> (none)
- SW79: renamed from SW78; value Down -> (none); footprint Button_Switch_Keyboard:SW_Cherry_MX_1.00u_PCB -> (none)
- SW8: value F6 -> (none); footprint Button_Switch_Keyboard:SW_Cherry_MX_1.00u_PCB -> (none)
- SW80: renamed from SW79; value Right -> (none); footprint Button_Switch_Keyboard:SW_Cherry_MX_1.00u_PCB -> (none)
- SW9: value F7 -> (none); footprint Button_Switch_Keyboard:SW_Cherry_MX_1.00u_PCB -> (none)
Connections:
- net COL 0A: now also SW75.2
- net ROW 05: now also D75.1 (K)
- new net: D75.2 (A), SW75.1
